File: e1_phy.sch (EAGLE design)
At the start: 53 parts, among them U1 XRT82D20, X1 RJ45-8L-B, X2 MINI-USB-32005-201

Commit message: First sane version, for review.
I've smashed all the random edits and redesigns into this single commit,
the history was not useful to keep.
Parts:
- removed X1: RJ45-8L-B, con-tycoelectronics:RJ45-8L-B
- added C12, C13, C14, C15, C16, C17, C18, C19, C20, C25, C26, C27, C28: 100n, rcl:C-EUC0603
- added C21, C22, C23, C24: 10uF, rcl:C-EUC0603
- added CN1: (no value), adafruit:USBMINIB
- added D1: MBR0520LT, diode:MBR0520LT
- added IC1: (no value), linear:2AMP_P8+4D
- added IC2, IC3: LD117AS33TR, v-reg:LD117AS33TR
- added IC4: MCP4725, dp_devices:IC_MCP4725
- added L1: 10uH, rcl:L-EUL1812
- added LED3, LED4, LED5, LED6, LED7, LED8: (no value), led:LEDCHIPLED_0603
- added R30, R31: 33R, rcl:R-EU_R0603
- added R32: 27k, rcl:R-EU_R0603
- added R33: 47k, rcl:R-EU_R0603
- added R34, R50: DNP, rcl:R-EU_R0603
- added R35: 680k, rcl:R-EU_R0603
- added R36, R37, R38, R39, R40, R41: 10k, rcl:R-EU_R0603
- added R42: 0R (DNP), rcl:R-EU_R0603
- added R43, R44: BLM/0R, rcl:R-EU_R0603
- added R45: 0R, rcl:R-EU_R0603
- added R46: 1R, rcl:R-EU_R0603
- added R47, R48, R49, R51, R52, R53, R54, R55: 1k, rcl:R-EU_R0603
- added SV1, SV6: (no value), con-lstb:MA05-2
- added SV2, SV5: (no value), con-lstb:MA05-1
- added SV3: (no value), con-lstb:MA04-1
- added SV4: (no value), con-lstb:MA08-2
- added TP10, TP11, TP12, TP13, TP14, TP15, TP16, TP17, TP18, TP19, TP6, TP7, TP8, TP9: TPB1,27, testpad:TPB1,27
- added U2: GPS_GNS_2201, cvogel:GPS_GNS_2201
- added U3: VCTCXO-CONNORWINFIELD, Connor-Winfield_VCTCXO:VCTCXO-CONNORWINFIELD
- added U4: VCXO_TAITIEN_VT, cvogel:VCXO_TAITIEN_VT
- added X3: JACK2.5_SJ-2523, SJ-2523-JACK:JACK2.5_SJ-2523
- added X4: 0446200002, con-molex:0446200002
- C1, C10, C11, C2, C3, C4, C5, C6, C7, C8, C9: device rcl:C-EUC0805 -> rcl:C-EUC0603
- LED1, LED2: device led:LEDCHIP-LED0805 -> led:LEDCHIPLED_0603
- R1, R10, R11, R12, R16, R17, R18, R19, R2, R20, R21, R22, R23, R24, R25, R26, R27, R28, R29, R8, R9: device rcl:R-EU_R0805 -> rcl:R-EU_R0603
- R13: value 0R -> DNP; device rcl:R-EU_R0805 -> rcl:R-EU_R0603
- R14: value DNP -> 10k; device rcl:R-EU_R0805 -> rcl:R-EU_R0603
- R15: value ? -> 10k; device rcl:C-EUC0805 -> rcl:R-EU_R0603
- R3, R4, R5, R6: value 60R -> DNP; device rcl:R-EU_R0805 -> rcl:R-EU_R0603
- R7: value 0R -> 10k; device rcl:R-EU_R0805 -> rcl:R-EU_R0603
- X2: value MINI-USB-32005-201 -> SMA-142-0701-801/806; device con-cypressindustries:MINI-USB-32005-201 -> con-coax:SMA-142-0701-801/806
Connections:
- removed net N$3: R29.1, U1.TNEG_CODE
- removed net RX_SEC_CTR: R13.1, TR1A.SEC_2
- new net #GPS_RESET: TP18.TP, U2.#RESET
- new net #RESET: SV1.10, U$1.NRST
- new net #SPI_CS0: SV6.5, U$1.PA11
- new net #SPI_CS1: SV6.6, U$1.PA30
- new net +UB: C15.1, C20.1, C24.1, C25.2, C26.2, C27.2, C28.2, IC1P.V+, IC3.OUT, IC4.3, R40.1, R47.2, SV5.5, U$1.ADVREF, U3.VCC, U4.VCC
- new net +UB_HALF: C16.2, IC1A.+IN, IC1B.+IN, R40.2, R41.2
- new net DAC0: R36.1, U$1.PB13_DAC0
- new net DAC1: R35.1, U$1.PB14_DAC1
- new net DAC_I2C: IC4.1, R15.1
- new net GPS_PPS: SV2.2, U$1.PA0, U2.1PPS
- new net GPS_SAM4_RX: SV2.3, U$1.PA5, U2.TX_A
- new net GPS_SAM4_TX: SV2.4, U$1.PA6, U2.RX_A
- new net I2C_SCL: IC4.5, SV6.8, U$1.PA4
- new net I2C_SDA: IC4.4, SV6.7, U$1.PA3
- new net JTAGSEL: R45.2, U$1.JTAGSEL
- new net LED1: R51.2, U$1.PA24
- new net LED2: R52.2, U$1.PA25
- new net LED3: R53.2, U$1.PA26
- new net LINE_PIN3: R3.2, X4.3
- new net LINE_PIN6: R4.2, X4.6
- new net LINE_PIN7: R5.2, X4.7
- new net LINE_PIN8: R6.2, X4.8
- new net N$10: R49.2, U2.3D_FIX
- new net N$11: LED5.A, R49.1
- new net N$12: CN1.VBUS, D1.A, R32.2
- new net N$13: C19.1, IC3.IN, R44.1
- new net N$14: C17.1, IC2.IN, R43.1
- new net N$15: C21.1, R46.1
- new net N$16: LED3.A, R47.1
- new net N$17: TP16.TP, U$1.PA29
- new net N$18: LED4.A, R48.1
- new net N$19: TP12.TP, U$1.PA23
- new net N$20: TP13.TP, U$1.PA15
- new net N$21: TP7.TP, U$1.PB2_AD6
- new net N$22: TP14.TP, U$1.PA27
- new net N$23: TP15.TP, U$1.PA28
- new net N$24: TP19.TP, U2.WAKEUP
- new net N$26: LED6.A, R51.1
- new net N$27: LED7.A, R52.1
- new net N$28: LED8.A, R53.1
- new net N$4: U2.RF_IN, X2.1
- new net OPAMP1_IN_NEG: C14.1, IC1A.-IN, R15.2, R35.2, R36.2, R38.1, R42.1
- new net OPAMP1_OUT: C14.2, IC1A.OUT, R37.1, R38.2
- new net OPAMP2_IN_NEG: C13.1, IC1B.-IN, R37.2, R39.1
- new net PB12_ERASE: R13.2, U$1.PB12_ERASE
- new net SAM4S_CLK: SV5.4, U$1.PB9_XIN, U3.FO, U4.Q
- new net SPI_MISO: SV6.3, U$1.PA12
- new net SPI_MOSI: SV6.4, U$1.PA13
- new net SPI_SCK: SV6.1, U$1.PA14
- new net TCK_SWDCLK: SV1.4, U$1.PB7_TCK_SWCLK
- new net TDI: SV1.8, U$1.PB4_TDI
- new net TDO: SV1.6, U$1.PB5_TDO
- new net TMS_SWDIO: SV1.2, U$1.PB6_TMS_SWDIO
- new net TNEG_CODE: R29.1, SV4.9, U1.TNEG_CODE
- new net TST: R34.2, U$1.TST
- new net URXD0_SAMBA_RX: SV3.3, U$1.PA9, X3.TIP
- new net USB_DDM: R31.1, U$1.PB10_DDM
- new net USB_DDM_CON: CN1.D-, R31.2
- new net USB_DDP: R30.1, U$1.PB11_DDP
- new net USB_DDP_CON: CN1.D+, R30.2
- new net USB_VBUS_CON: D1.C, R43.2, R44.2
- new net USB_VBUS_SENS: R32.1, R33.2
- new net UTXD0_SAMBA_TX: SV3.2, U$1.PA10, X3.MIDDLE
- new net VCTCXO_EN: R14.1, U$1.PB0_AD4, U3.OE
- new net VCXO_CTRL: C13.2, IC1B.OUT, R39.2, R42.2, SV5.2, U3.CV, U4.VADJ
- new net VCXO_EN: R7.2, SV5.3, U$1.PB1_AD5, U4.OE
- new net VDDCORE: C10.1, C11.1, C22.1, C9.1, L1.2, U$1.VDDCORE, U$1.VDDOUT
- new net VDDPLL: C8.1, L1.1, R46.2, U$1.VDDPLL
- net #CLKLOS: now also SV4.8, U$1.PA8_XOUT32
- net #DLOOP: now also SV4.10
- net #LLOOP: now also SV4.12
- net #RLOOP: now also SV4.11
- net #RLOS: now also SV4.7, U$1.PA7_XIN32
- net CLK2048: now also SV4.16, U$1.PA21_AD8
- net GND: now also C12.2, C15.2, C16.1, C17.2, C18.2, C19.2, C20.2, C21.2, C22.2, C23.2, C24.2, C25.1, C26.1, C27.1, C28.1, CN1.GND, IC1P.V-, IC2.ADJ, IC3.ADJ, IC4.2, IC4.6, LED3.C, LED4.C, LED5.C, LED6.C, LED7.C, LED8.C, R33.1, R41.1, R50.2, R7.1, SV1.3, SV1.5, SV1.9, SV2.1, SV3.1, SV4.15, SV4.2, SV5.1, SV6.2, SV6.9, TR1A.SEC_2, U2.GND, U2.RF_GND, U3.GND, U4.GND, X2.2, X3.RING; no longer R13.2, R15.2
- net GNDIO: now also R3.1, R4.1, R5.1, R50.1, R6.1, TP6.TP, X4.S1, X4.S2; no longer R14.1, R15.1, R7.2
- net JAEN: now also R54.2, SV4.14
- net JATX: now also R55.2, SV4.13
- net LINE_PIN1: now also X4.1; no longer X1.1
- net LINE_PIN2: now also X4.2; no longer X1.2
- net LINE_PIN4: now also X4.4; no longer X1.4
- net LINE_PIN5: now also X4.5; no longer X1.5
- net N$5: now also TP17.TP, U$1.PA31; no longer R3.2, X1.3
- net N$6: now also TP9.TP, U$1.PA2; no longer R4.2, X1.6
- net N$7: now also TP8.TP, U$1.PA1; no longer R5.2, X1.7
- net N$8: now also TP10.TP, U$1.PA20_AD3; no longer R6.2, X1.8
- net N$9: now also TP11.TP, U$1.PA22_AD9; no longer R3.1, R4.1, R5.1, R6.1, R7.1
- net RX_CLK: now also SV4.3, U$1.PA19_AD2
- net RX_DATA: now also SV4.1, U$1.PA18_AD1
- net RX_VIOLATION: now also SV4.4
- net TX_CLK: now also SV4.5, U$1.PA16, U$1.PB3_AD7
- net TX_DATA: now also SV4.6, U$1.PA17_AD0
- net VCC: now also C12.1, C18.1, C23.1, IC2.OUT, R13.1, R34.1, R45.1, R48.2, R54.1, R55.1, SV1.1, SV2.5, SV3.4, SV6.10, U$1.VDDIN, U2.VBACKUP, U2.VCC; no longer C10.1, C11.1, C8.1, C9.1, U$1.VDDCORE
Other:
- note added: ""Clean" supply"
- note added: ""GNDIO" is intended for debugging, e.g. for connecting a scope. Do not populate Rs for production."
- note added: "1kHz"
- note added: "ATSAM4S-2B: 128k/64k -4B: 256/64, -8B: 512/128 -16B 1024/128"
- note added: "Bypass if OpAmp and associated components are not populated."
- note added: "JAEN&JATX int pd ext pu to enable and put in TX path RAOS int pd: disable receive all ones TAOS int pd: disable transmit all ones"
- note added: "JTAG/SWD"
- note added: "JTAGSEL: enable JTAG/SWD TST: disable prog. mode"
- note added: "LUI Signals"
- note added: "OSMOCOM Standard Serial Cable Tip: PC to Device Ring: Device to PC Sleeve: GND"
- note added: "PCB size 100mm x 75mm, Fischer FR-80-42-100-ME"
- note added: "SPI and I2C"
- note added: "Status/Debugging LEDs"
- note added: "Usb Rext=27R on eval"
- note added: "VCXO clk, enable, ctrl voltage"
- note added: "analog summing DAC+DAC1/x summing junction kept at +UB/2"
- note added: "e1_sam4_usb vogelchr@vogel.cx 2018-06-24 for review"
- note added: "external GPS"
- note removed: "3 or 6 used for Rx/Tx shield"
- note removed: "GNDIO / GND Plane Separation"
- note removed: "RAOS int pd: disable receive all ones TAOS int pd: disable transmit all ones"
- moved on the sheet: C10, C11, C8, C9, R13, R14, R15, R18, R19, R29, R7, TP3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
