File: e1_phy.sch (EAGLE design)
At the start: 145 parts, among them IC2 LD117AS33TR, IC3 LD117AS33TR, IC4 MAX6173AASA, U1 IDT82V2081, U2 GPS_GNS_2201, U3 VCTCXO-CONNORWINFIELD, U4 VCXO_TAITIEN_VT, U5 IP4234CZ6, U7 IP4234CZ6, X1 BU-SMA-G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

Commit message: Some cleanup before declaring final.
ADVREF of SAM4S fed by VREF net.
+UB/2 divider fed by VREF net, renamed to VREF_HALF.
Parts:
- added TP17: TPB1,27, testpad:TPB1,27
Connections:
- net +UB_HALF renamed VREF_HALF
- removed net N$7: IC4.OUT, R23.1, TP6.TP, U6.REF
- new net TP17: TP17.TP, U$1.PB8_XOUT
- new net VREF: C26.2, IC4.OUT, R23.1, R40.1, TP6.TP, U$1.ADVREF, U6.REF
- net +UB: no longer C26.2, R40.1, U$1.ADVREF
Other:
- note added: "e1_sam4_usb vogelchr@vogel.cx 2018-07-09 final"
- note removed: "e1_sam4_usb vogelchr@vogel.cx 2018-07-03 for review"
Changed lines of the file:
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@@
 <part name="GND21" library="supply1" library_urn="urn:adsk.eagle:library:371" deviceset="GND" device=""/>
 <part name="GND22" library="supply1" library_urn="urn:adsk.eagle:library:371" deviceset="GND" device=""/>
-<part name="SUPPLY3" library="supply2" library_urn="urn:adsk.eagle:library:372" deviceset="+UB" device=""/>
 <part name="L1" library="rcl" library_urn="urn:adsk.eagle:library:334" deviceset="L-EU" device="L1812" package3d_urn="urn:adsk.eagle:package:23494/2" value="10uH"/>
 <part name="C21" library="rcl" library_urn="urn:adsk.eagle:library:334" deviceset="C-EU" device="C0603" package3d_urn="urn:adsk.eagle:package:23616/2" value="10uF"/>
@@
 <part name="TP5" library="testpad" library_urn="urn:adsk.eagle:library:385" deviceset="TP" device="B1,27" package3d_urn="urn:adsk.eagle:package:27944/1"/>
 <part name="TP6" library="testpad" library_urn="urn:adsk.eagle:library:385" deviceset="TP" device="B1,27" package3d_urn="urn:adsk.eagle:package:27944/1"/>
+<part name="TP17" library="testpad" library_urn="urn:adsk.eagle:library:385" deviceset="TP" device="B1,27" package3d_urn="urn:adsk.eagle:package:27944/1"/>
 </parts>
 <sheets>
@@
 <text x="289.56" y="25.4" size="2.1844" layer="97" font="fixed">e1_sam4_usb
 vogelchr@vogel.cx
-2018-07-03 for review</text>
+2018-07-09 final</text>
 <text x="292.1" y="45.72" size="1.778" layer="97">FTDI Pinout
 2=#CTS
@@
 <instance part="C15" gate="G$1" x="320.04" y="157.48"/>
 <instance part="R39" gate="G$1" x="302.26" y="185.42"/>
-<instance part="SUPPLY1" gate="G$1" x="312.42" y="167.64"/>
+<instance part="SUPPLY1" gate="G$1" x="322.58" y="167.64"/>
 <instance part="R40" gate="G$1" x="304.8" y="162.56" rot="R180"/>
 <instance part="R41" gate="G$1" x="297.18" y="154.94" rot="R90"/>
@@
 <instance part="GND21" gate="1" x="12.7" y="149.86"/>
 <instance part="GND22" gate="1" x="12.7" y="132.08"/>
-<instance part="SUPPLY3" gate="G$1" x="63.5" y="180.34"/>
 <instance part="L1" gate="G$1" x="55.88" y="139.7" rot="R180"/>
 <instance part="C21" gate="G$1" x="40.64" y="127"/>
@@
 <instance part="TP5" gate="G$1" x="269.24" y="55.88" rot="R270"/>
 <instance part="TP6" gate="G$1" x="208.28" y="167.64"/>
+<instance part="TP17" gate="G$1" x="104.14" y="208.28"/>
 </instances>
 <busses>
@@
 <segment>
 <pinref part="C15" gate="G$1" pin="1"/>
-<pinref part="R40" gate="G$1" pin="1"/>
-<wire x1="309.88" y1="162.56" x2="312.42" y2="162.56" width="0.1524" layer="91"/>
-<wire x1="312.42" y1="162.56" x2="314.96" y2="162.56" width="0.1524" layer="91"/>
 <wire x1="314.96" y1="162.56" x2="320.04" y2="162.56" width="0.1524" layer="91"/>
 <wire x1="320.04" y1="162.56" x2="320.04" y2="160.02" width="0.1524" layer="91"/>
 <pinref part="IC1" gate="P" pin="V+"/>
 <wire x1="314.96" y1="160.02" x2="314.96" y2="162.56" width="0.1524" layer="91"/>
-<junction x="314.96" y="162.56"/>
 <pinref part="SUPPLY1" gate="G$1" pin="+UB"/>
-<wire x1="312.42" y1="165.1" x2="312.42" y2="162.56" width="0.1524" layer="91"/>
-<junction x="312.42" y="162.56"/>
+<wire x1="322.58" y1="165.1" x2="322.58" y2="162.56" width="0.1524" layer="91"/>
+<wire x1="322.58" y1="162.56" x2="320.04" y2="162.56" width="0.1524" layer="91"/>
+<junction x="320.04" y="162.56"/>
 </segment>
 <segment>
@@
 </segment>
 <segment>
-<pinref part="U$1" gate="G$1" pin="ADVREF"/>
-<pinref part="SUPPLY3" gate="G$1" pin="+UB"/>
-<wire x1="68.58" y1="175.26" x2="63.5" y2="175.26" width="0.1524" layer="91"/>
-<wire x1="63.5" y1="175.26" x2="63.5" y2="177.8" width="0.1524" layer="91"/>
-<pinref part="C26" gate="G$1" pin="2"/>
-<wire x1="60.96" y1="175.26" x2="63.5" y2="175.26" width="0.1524" layer="91"/>
-<junction x="63.5" y="175.26"/>
-</segment>
-<segment>
 <pinref part="SUPPLY4" gate="G$1" pin="+UB"/>
 <wire x1="10.16" y1="198.12" x2="10.16" y2="195.58" width="0.1524" layer="91"/>
@@
 </segment>
 </net>
-<net name="+UB_HALF" class="0">
+<net name="VREF_HALF" class="0">
 <segment>
 <pinref part="IC1" gate="A" pin="+IN"/>
@@
 </segment>
 </net>
-<net name="N$7" class="0">
+<net name="VREF" class="0">
 <segment>
 <pinref part="IC4" gate="G$1" pin="OUT"/>
@@
 <wire x1="208.28" y1="165.1" x2="208.28" y2="162.56" width="0.1524" layer="91"/>
 <junction x="208.28" y="162.56"/>
+<label x="210.82" y="177.8" size="1.27" layer="95" rot="R90"/>
+</segment>
+<segment>
+<pinref part="U$1" gate="G$1" pin="ADVREF"/>
+<wire x1="68.58" y1="175.26" x2="66.04" y2="175.26" width="0.1524" layer="91"/>
+<pinref part="C26" gate="G$1" pin="2"/>
+<wire x1="66.04" y1="175.26" x2="60.96" y2="175.26" width="0.1524" layer="91"/>
+<wire x1="48.26" y1="185.42" x2="66.04" y2="185.42" width="0.1524" layer="91"/>
+<wire x1="66.04" y1="185.42" x2="66.04" y2="175.26" width="0.1524" layer="91"/>
+<junction x="66.04" y="175.26"/>
+<label x="48.514" y="185.674" size="1.27" layer="95"/>
+</segment>
+<segment>
+<pinref part="R40" gate="G$1" pin="1"/>
+<wire x1="309.88" y1="162.56" x2="312.42" y2="162.56" width="0.1524" layer="91"/>
+<wire x1="312.42" y1="162.56" x2="312.42" y2="170.18" width="0.1524" layer="91"/>
+<wire x1="312.42" y1="170.18" x2="320.04" y2="170.18" width="0.1524" layer="91"/>
+<label x="312.42" y="170.688" size="1.27" layer="95"/>
 </segment>
 </net>
@@
 </segment>
 </net>
+<net name="TP17" class="0">
+<segment>
+<pinref part="TP17" gate="G$1" pin="TP"/>
+<pinref part="U$1" gate="G$1" pin="PB8_XOUT"/>
+<wire x1="104.14" y1="205.74" x2="104.14" y2="195.58" width="0.1524" layer="91"/>
+<label x="103.632" y="196.342" size="1.27" layer="95" rot="R90"/>
+</segment>
+</net>
