File: e1_phy_v7.sch (EAGLE design)
At the start: 136 parts, among them IC2 LD117AS33TR, IC3 LD117AS33TR, IC4 MCP4725, U1 XRT82D20, U2 GPS_GNS_2201, U3 VCTCXO-CONNORWINFIELD, U4 VCXO_TAITIEN_VT, X2 SMA-142-0701-801/806, X3 JACK2.5_SJ-2523, X4 0446200002

Commit message: Pullup on i2c, ERASE jumper.
Parts:
- JP2: device jumper:JP1E -> jumper@1:JP1E
- SV4: device con-lstb:MA08-2 -> con-lstb@1:MA08-2
Changed lines of the file:
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@@
 <?xml version="1.0" encoding="utf-8"?>
 <!DOCTYPE eagle SYSTEM "eagle.dtd">
-<eagle version="9.0.1">
+<eagle version="7.7.0">
 <drawing>
 <settings>
@@
 <part name="GND1" library="supply1" deviceset="GND" device=""/>
 <part name="TP7" library="testpad" deviceset="TP" device="B1,27"/>
-<part name="SV4" library="con-lstb" library_urn="urn:adsk.eagle:library:162" deviceset="MA08-2" device="" package3d_urn="urn:adsk.eagle:package:8335/1"/>
+<part name="SV4" library="con-lstb@1" deviceset="MA08-2" device=""/>
 <part name="GND2" library="supply1" deviceset="GND" device=""/>
 <part name="GND16" library="supply1" deviceset="GND" device=""/>
@@
 <part name="TP18" library="testpad" deviceset="TP" device="B1,27"/>
 <part name="TP19" library="testpad" deviceset="TP" device="B1,27"/>
-<part name="X4" library="con-molex" library_urn="urn:adsk.eagle:library:165" deviceset="0446200002" device=""/>
+<part name="X4" library="con-molex" deviceset="0446200002" device=""/>
 <part name="GND30" library="supply1" deviceset="GNDIO" device=""/>
 <part name="R56" library="rcl" deviceset="R-EU_" device="R0603" value="10k"/>
 <part name="R57" library="rcl" deviceset="R-EU_" device="R0603" value="10k"/>
 <part name="P+4" library="supply1" deviceset="VCC" device=""/>
-<part name="JP2" library="jumper" library_urn="urn:adsk.eagle:library:252" deviceset="JP1E" device="" package3d_urn="urn:adsk.eagle:package:15455/1"/>
+<part name="JP2" library="jumper@1" deviceset="JP1E" device=""/>
 </parts>
 <sheets>
@@
 which will not be processed correctly with this version.
 </note>
-<note version="8.2" severity="warning">
-Since Version 8.2, EAGLE supports online libraries. The ids
-of those online libraries will not be understood (or retained)
-with this version.
-</note>
-<note version="8.3" severity="warning">
-Since Version 8.3, EAGLE supports URNs for individual library
-assets (packages, symbols, and devices). The URNs of those assets
-will not be understood (or retained) with this version.
-</note>
-<note version="8.3" severity="warning">
-Since Version 8.3, EAGLE supports the association of 3D packages
-with devices in libraries, schematics, and board files. Those 3D
-packages will not be understood (or retained) with this version.
-</note>
 </compatibility>

Commit message: Changed LIU to IDT82V2081.
Parts:
- removed LED1, LED2: (no value), led:LEDCHIPLED_0603
- removed R16, R17: 0R, rcl:R-EU_R0603
- removed R18, R19, R20, R24: DNP, rcl:R-EU_R0603
- removed R21, R22, R23, R29, R54, R55: 1k, rcl:R-EU_R0603
- removed SV4: (no value), con-lstb@1:MA08-2
- removed TP1, TP17, TP2, TP3, TP4, TP5, TP6: TPB1,27, testpad:TPB1,27
- added C29: 100n, rcl:C-EUC0603
- added D2, D3, D4, D5, D6, D7, D8, D9: MBR0520LT, diode@1:MBR0520LT
- added U$2: MNR 8x10k, laforge:MNR
- C3: value 10u -> 100n
- R10, R11: value 9R1 -> 10k
- R12: value DNP -> 10k
- R8: value 60R -> DNP
- R9: value 60R -> 3k 1%
- TR1: value PE-65861 -> PULSE_T1094NL; device cvogel:PULSE_PE65861 -> laforge:PULSE_T1094NL
- U1: value XRT82D20 -> IDT82V2081; device cvogel:XRT82D20 -> idt82v2081:IDT82V2081
Connections:
- removed net #ATM: R24.1, U1.#ATM
- removed net #CLKLOS: R23.1, SV4.8, U$1.PA8_XOUT32, U1.#CLKLOS
- removed net #DLOOP: SV4.10, U1.#DLOOP
- removed net #LLOOP: SV4.12, U1.#LLOOP
- removed net #RLOOP: SV4.11, U1.#RLOOP
- removed net #RLOS: R22.1, SV4.7, U$1.PA7_XIN32, U1.#RLOS
- removed net DIGI: R18.1, U1.DIGI
- removed net JAEN: R54.2, SV4.14, U1.JAEN
- removed net JATX: R55.2, SV4.13, U1.JATX_DR
- removed net MUTERX: R21.1, U1.MUTERX
- removed net N$1: LED1.C, R22.2
- removed net N$2: LED2.C, R23.2
- removed net RAOS: R19.2, U1.RAOS
- removed net RRING_LIU: R17.2, TP2.TP, U1.RRING
- removed net RTIP_LIU: R16.2, TP1.TP, U1.RTIP
- removed net RX_PRI_CTR: R1.2, TR1A.PRI_2
- removed net RX_VIOLATION: SV4.4, U1.RNEG_LCV
- removed net TAOS: R20.2, U1.TAOS
- removed net TNEG_CODE: R29.1, SV4.9, U1.TNEG_CODE
- removed net TRING_XFMR: R11.1, TR1B.PRI_3
- removed net TTIP_XFMR: R10.1, TR1B.PRI_1
- removed net TX_PRI_CTR: R12.1, TR1B.PRI_2
- removed net TX_SEC_CTR: R2.2, TR1B.SEC_2
- new net #RST_LIU: U$1.PA8_XOUT32, U1.#RST
- new net #SPI_CS2: R11.1, SV6.6, U$1.PA30
- new net AD0: U$2.8, U1.AD0_PATT0
- new net AD1: U$2.4, U1.AD1/PATT1
- new net AD2: U$2.7, U1.AD2/RPD
- new net AD3: U$2.3, U1.AD3/EQ
- new net AD4: U$2.6, U1.AD4/PULS0
- new net AD5: U$2.2, U1.AD5/PULS1
- new net AD6: U$2.5, U1.AD6/PULS2
- new net AD7: U$2.1, U1.AD7/PULS3
- new net LOS_LIU: U$1.PA7_XIN32, U1.LOS
- new net N$25: R8.2, TR1-1:2.P$6
- new net N$31: R9.1, U1.R_REF
- net #SPI_CS0: now also R10.1
- net #SPI_CS1: now also R12.2, U$1.PA31, U1.#CS/RXTX1; no longer SV6.6, U$1.PA30
- net +UB: now also C29.1, U1.VDDA
- net CLK2048: no longer SV4.16
- net E1_LINE_RX_A: now also TR1-1:1.P$1; no longer TR1A.PRI_1
- net E1_LINE_RX_B: now also TR1-1:1.P$3; no longer TR1A.PRI_3
- net E1_LINE_TX_A: now also TR1-1:2.P$1; no longer TR1B.SEC_1
- net E1_LINE_TX_B: now also TR1-1:2.P$3; no longer TR1B.SEC_3
- net GND: now also C29.2, D6.A, D7.A, D8.A, D9.A, U$2.C, U$2.D, U1.GNDA, U1.GNDD, U1.GNDIO, U1.GNDT, U1.IC2_GND, U1.JA0, U1.JA1, U1.MODE1, U1.RCLKE, U1.SCLKE/#RD/#DS/MONT, U1.TDN, U1.THZ; no longer R12.2, R24.2, R8.2, SV4.15, SV4.2, TP5.TP, TR1A.SEC_2, U1.AGND, U1.TGND, U1.TXLEV
- net GNDIO: no longer R1.1, R2.1, TP6.TP
- net N$5: now also R2.2, TR1-1:2.P$4; no longer TP17.TP, U$1.PA31
- net RRING: now also D3.A, D7.C, R1.2, TR1-1:1.P$6, U1.RRING; no longer R17.1, R9.1, TR1A.SEC_3
- net RTIP: now also D2.A, D6.C, R1.1, TR1-1:1.P$4, U1.RTIP; no longer R16.1, R8.1, TR1A.SEC_1
- net RX_CLK: no longer SV4.3
- net RX_DATA: now also U1.RD_RDP; no longer SV4.1, U1.RPOS_RDATA
- net SPI_MISO: now also U1.SDO/#ACK/RDY/TERM
- net SPI_MOSI: now also U1.SDI/#WR/R#W/LP0
- net SPI_SCK: now also U1.SCLK/ALE/AS/LP1
- net TRING: now also D5.A, D9.C, R8.1; no longer R11.2, TP4.TP
- net TTIP: now also D4.A, D8.C, R2.1; no longer R10.2, TP3.TP
- net TX_CLK: no longer SV4.5
- net TX_DATA: now also U1.TD_TDP; no longer SV4.6, U1.TPOS_TDATA
- net VCC: now also D2.C, D3.C, D4.C, D5.C, R10.2, R11.2, R12.1, U1.MODE0, U1.VDDD, U1.VDDIO, U1.VDDT; no longer LED1.A, LED2.A, R18.2, R19.1, R20.1, R21.2, R29.2, R54.1, R55.1, U1.AVDD, U1.TVDD
Other:
- note added: "1"
- note added: "16-14=PRI PRI:SEC=1:1"
- note added: "2"
- note added: "6-8=PRI PRI:SEC=1:2"
- note added: "e1_sam4_usb vogelchr@vogel.cx 2018-06-25 for review"
- note removed: "JAEN&JATX int pd ext pu to enable and put in TX path RAOS int pd: disable receive all ones TAOS int pd: disable transmit all ones"
- note removed: "LUI Signals"
- note removed: "Line:LIU Rx 1:2"
- note removed: "Line:LIU Tx 2:1"
- note removed: "MuteRX ext pullup: enable #ClkLOS=0 RCLK=1, RDATA=0 DIGI: int. pulldn: xDATA high active TNEG ext pullup: int. HDB3 enc/decoder #ATM int pullup: alarm test mode inactive"
- note removed: "e1_sam4_usb vogelchr@vogel.cx 2018-06-24 for review"
- note removed: "line side R should probably *never* be populated!"
- moved on the sheet: C1, C2, C3, R1, R10, R11, R12, R2, R8, R9

Commit message: Regenerated v7 eagle files, made .pdf for schematic.
 -> next release candidate 20180703
Parts:
- removed IC4: MCP4725, dp_devices:IC_MCP4725
- removed R32: 27k, rcl:R-EU_R0603
- removed R33: 47k, rcl:R-EU_R0603
- removed R56, R57: 10k, rcl:R-EU_R0603
- removed SV6: (no value), con-lstb:MA05-2
- removed U$2: MNR 8x10k, laforge:MNR
- added D10: 0603ESDA-TR, laforge:0603ESDA-TR
- added L2: 10uH, rcl:L-EUL1812
- added RN1, RN2: (no value), resistor-dil:4R-NEXB38V
- added RN3, RN4: 10k, resistor-dil:4R-NEXB38V
- added SV4: (no value), con-lstb@1:MA06-1
- added U5, U7: IP4234CZ6, laforge:IP4234CZ6
- added U6: (no value), max5215_max5217:MAX521X
- R1: value DNP -> 120R
- R2, R8: value DNP -> 9R
- SV1: device con-lstb:MA05-2 -> con-lstb@1:MA05-2
- SV3: device con-lstb:MA04-1 -> con-lstb@1:MA10-2
Connections:
- net USB_VBUS_CON renamed USB_VBUS
- removed net LOS_LIU: U$1.PA7_XIN32, U1.LOS
- removed net N$12: CN1.VBUS, D1.A, R32.2
- removed net USB_VBUS_SENS: R32.1, R33.2
- new net #LIU_INT: U$1.PA7_XIN32, U1.#INT/RXTXM0
- new net LIU_VDDA: C29.1, L2.2, U1.VDDA
- new net N$1: CN1.D+, U5.1A
- new net N$2: CN1.D-, U5.2A
- new net N$32: SV4.2, SV4.6
- new net URXD0_SAMBA_RX_CON: R10.1, SV4.4, U7.2A, X3.TIP
- new net UTXD0_SAMBA_TX_CON: SV4.5, U7.1A, X3.MIDDLE
- new net VBUS_CONN: CN1.VBUS, D1.A, U5.VCC
- net #RESET: now also RN4D.1, SV3.15; no longer SV1.10
- net #RST_LIU: now also R11.1
- net #SPI_CS0: now also RN3B.1, SV1.10; no longer R10.1, SV6.5
- net #SPI_CS2: now also RN3D.1, SV1.4; no longer R11.1, SV6.6
- net +UB: now also U6.REF, U6.VDD; no longer C29.1, IC4.3, U1.VDDA
- net AD0: now also RN2A.2; no longer U$2.8
- net AD1: now also RN2B.2; no longer U$2.4
- net AD2: now also RN2C.2; no longer U$2.7
- net AD3: now also RN2D.2; no longer U$2.3
- net AD4: now also RN1D.1; no longer U$2.6
- net AD5: now also RN1C.1; no longer U$2.2
- net AD6: now also RN1B.1; no longer U$2.5
- net AD7: now also RN1A.1; no longer U$2.1
- net DAC_I2C: now also U6.OUT; no longer IC4.1
- net GND: now also D10.K, RN1A.2, RN1B.2, RN1C.2, RN1D.2, RN2A.1, RN2B.1, RN2C.1, RN2D.1, SV1.2, SV3.10, SV3.12, SV3.14, SV3.16, SV3.18, SV3.20, SV3.4, SV3.6, SV3.8, SV4.1, U5.GND, U6.GND, U7.GND; no longer IC4.2, IC4.6, R33.1, SV1.3, SV1.5, SV1.9, SV3.1, SV6.2, SV6.9, U$2.C, U$2.D
- net I2C_SCL: now also RN3C.1, SV1.5, U6.SCL; no longer IC4.5, R57.1, SV6.8
- net I2C_SDA: now also RN3A.1, SV1.6, U6.SDA; no longer IC4.4, R56.1, SV6.7
- net N$4: now also D10.A
- net SPI_MISO: now also SV1.7; no longer SV6.3
- net SPI_MOSI: now also SV1.8; no longer SV6.4
- net SPI_SCK: now also SV1.9; no longer SV6.1
- net TCK_SWDCLK: now also RN4B.1, SV3.9; no longer SV1.4
- net TDI: now also SV3.5; no longer SV1.8
- net TDO: now also SV3.13; no longer SV1.6
- net TMS_SWDIO: now also RN4A.1, SV3.7; no longer SV1.2
- net URXD0_SAMBA_RX: now also U7.2B; no longer SV3.3, X3.TIP
- net USB_DDM_CON: now also U5.2B; no longer CN1.D-
- net USB_DDP_CON: now also U5.1B; no longer CN1.D+
- net UTXD0_SAMBA_TX: now also U7.1B; no longer SV3.2, X3.MIDDLE
- net VCC: now also L2.1, RN3A.2, RN3B.2, RN3C.2, RN3D.2, RN4A.2, RN4B.2, RN4C.2, RN4D.2, SV3.1, U7.VCC; no longer R56.2, R57.2, SV3.4, SV6.10
Other:
- note added: "FTDI Pinout 2=#CTS 6=#RTS 3=VCC"
- note added: "Power LEDs"
- note added: "UEXT 4="TxD"=#CS2"
- note added: "e1_sam4_usb vogelchr@vogel.cx 2018-07-03 for review"
- note removed: "SPI and I2C"
- note removed: "e1_sam4_usb vogelchr@vogel.cx 2018-06-25 for review"
- moved on the sheet: C1, C10, C11, C17, C18, C19, C2, C20, C21, C22, C23, C24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

Commit message: Testpads for unused LIU signals.
Parts:
- removed X2: SMA-142-0701-801/806, con-coax:SMA-142-0701-801/806
- added C30: 100n, rcl:C-EUC0603
- added IC4: MAX6173AASA, maxim:MAX6173AASA
- added R16, R17, R18, R19, R20, R21, R22: 33R, rcl:R-EU_R0603
- added R23: 0R (DNP), rcl:R-EU_R0603
- added R24: BLM/0R, rcl:R-EU_R0603
- added R29: 10k, rcl:R-EU_R0603
- added TP1, TP2, TP3: TPB1,27, testpad:TPB1,27
- added X1: BU-SMA-G, con-coax:BU-SMA-G
Connections:
- net N$10 renamed GPS_3DFIX
- net N$19 renamed TP12
- net N$20 renamed TP13
- net N$21 renamed TP7
- net N$22 renamed TP14
- net N$23 renamed TP15
- net N$24 renamed GPS_WAKEUP
- net N$6 renamed TP9
- net N$7 renamed TP8
- net N$8 renamed TP10
- net N$9 renamed TP11
- new net CLK2048_SAM4S: R19.1, U$1.PA21_AD8
- new net GPS_RF: D10.A, U2.RF_IN, X1.1
- new net GPS_RX_A: R20.2, U2.RX_A
- new net N$30: R22.2, U2.1PPS
- new net N$6: R29.2, TP1.TP, U1.TDN
- new net N$7: IC4.OUT, R23.1, U6.REF
- new net N$8: TP3.TP, U1.LOS
- new net N$9: C30.2, IC4.IN, R24.2
- new net SAM4S_CLK_EXT: R18.2, SV5.4
- new net SAM4S_CLK_VCTXO: R17.2, U3.FO
- new net SAM4S_CLK_VCXO: R16.2, U4.Q
- new net TPS_TX_A: R21.2, U2.TX_A
- net +UB: now also R23.2; no longer U6.REF
- net CLK2048: now also R19.2; no longer U$1.PA21_AD8
- net GND: now also C30.1, IC4.GND, R29.1, X1.2; no longer U1.TDN, X2.2
- net GPS_PPS: now also R22.1, SV2.4; no longer SV2.2, U2.1PPS
- net GPS_SAM4_RX: now also R21.1; no longer U2.TX_A
- net GPS_SAM4_TX: now also R20.1, SV2.2; no longer SV2.4, U2.RX_A
- net N$4: now also TP2.TP, U1.CV_RDN; no longer D10.A, U2.RF_IN, X2.1
- net SAM4S_CLK: now also R16.1, R17.1, R18.1; no longer SV5.4, U3.FO, U4.Q
- net USB_VBUS: now also R24.1
Other:
- note added: "use MAX6163"
- moved on the sheet: R14, SV5

Commit message: Cleaned up silkscreen.
Parts:
- added TP4, TP5, TP6: TPB1,27, testpad:TPB1,27
Connections:
- net CLK2048: now also TP4.TP
- net N$7: now also TP6.TP
- net TX_CLK: now also TP5.TP
Changed lines of the file:
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@@
 <part name="R29" library="rcl" deviceset="R-EU_" device="R0603" value="10k"/>
 <part name="TP3" library="testpad" deviceset="TP" device="B1,27"/>
+<part name="TP4" library="testpad" deviceset="TP" device="B1,27"/>
+<part name="TP5" library="testpad" deviceset="TP" device="B1,27"/>
+<part name="TP6" library="testpad" deviceset="TP" device="B1,27"/>
 </parts>
 <sheets>
@@
 <instance part="R29" gate="G$1" x="276.86" y="58.42" rot="R180"/>
 <instance part="TP3" gate="G$1" x="271.78" y="35.56" rot="R270"/>
+<instance part="TP4" gate="G$1" x="276.86" y="45.72"/>
+<instance part="TP5" gate="G$1" x="269.24" y="55.88" rot="R270"/>
+<instance part="TP6" gate="G$1" x="208.28" y="167.64"/>
 </instances>
 <busses>
@@
 <segment>
 <pinref part="U1" gate="G$1" pin="MCLK"/>
-<wire x1="254" y1="40.64" x2="266.7" y2="40.64" width="0.1524" layer="91"/>
-<label x="254.254" y="40.894" size="1.27" layer="95"/>
+<label x="277.114" y="40.894" size="1.27" layer="95"/>
+<wire x1="254" y1="40.64" x2="276.86" y2="40.64" width="0.1524" layer="91"/>
+<pinref part="TP4" gate="G$1" pin="TP"/>
+<wire x1="276.86" y1="40.64" x2="284.48" y2="40.64" width="0.1524" layer="91"/>
+<wire x1="276.86" y1="43.18" x2="276.86" y2="40.64" width="0.1524" layer="91"/>
+<junction x="276.86" y="40.64"/>
 </segment>
 </net>
@@
 <wire x1="254" y1="55.88" x2="266.7" y2="55.88" width="0.1524" layer="91"/>
 <label x="254.254" y="56.134" size="1.27" layer="95"/>
+<pinref part="TP5" gate="G$1" pin="TP"/>
 </segment>
 <segment>
@@
 <wire x1="210.82" y1="210.82" x2="210.82" y2="162.56" width="0.1524" layer="91"/>
 <junction x="210.82" y="162.56"/>
-</segment>
-</net>
+<pinref part="TP6" gate="G$1" pin="TP"/>
+<wire x1="208.28" y1="165.1" x2="208.28" y2="162.56" width="0.1524" layer="91"/>
+<junction x="208.28" y="162.56"/>
+</segment>
+</net>

Commit message: Some cleanup before declaring final.
ADVREF of SAM4S fed by VREF net.
+UB/2 divider fed by VREF net, renamed to VREF_HALF.
Parts:
- added TP17: TPB1,27, testpad:TPB1,27
Connections:
- net +UB_HALF renamed VREF_HALF
- removed net N$7: IC4.OUT, R23.1, TP6.TP, U6.REF
- new net TP17: TP17.TP, U$1.PB8_XOUT
- new net VREF: C26.2, IC4.OUT, R23.1, R40.1, TP6.TP, U$1.ADVREF, U6.REF
- net +UB: no longer C26.2, R40.1, U$1.ADVREF
Other:
- note added: "e1_sam4_usb vogelchr@vogel.cx 2018-07-09 final"
- note removed: "e1_sam4_usb vogelchr@vogel.cx 2018-07-03 for review"
Changed lines of the file:
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@@
 <part name="GND21" library="supply1" deviceset="GND" device=""/>
 <part name="GND22" library="supply1" deviceset="GND" device=""/>
-<part name="SUPPLY3" library="supply2" deviceset="+UB" device=""/>
 <part name="L1" library="rcl" deviceset="L-EU" device="L1812" value="10uH"/>
 <part name="C21" library="rcl" deviceset="C-EU" device="C0603" value="10uF"/>
@@
 <part name="TP5" library="testpad" deviceset="TP" device="B1,27"/>
 <part name="TP6" library="testpad" deviceset="TP" device="B1,27"/>
+<part name="TP17" library="testpad" deviceset="TP" device="B1,27"/>
 </parts>
 <sheets>
@@
 <text x="289.56" y="25.4" size="2.1844" layer="97" font="fixed">e1_sam4_usb
 vogelchr@vogel.cx
-2018-07-03 for review</text>
+2018-07-09 final</text>
 <text x="292.1" y="45.72" size="1.778" layer="97">FTDI Pinout
 2=#CTS
@@
 <instance part="C15" gate="G$1" x="320.04" y="157.48"/>
 <instance part="R39" gate="G$1" x="302.26" y="185.42"/>
-<instance part="SUPPLY1" gate="G$1" x="312.42" y="167.64"/>
+<instance part="SUPPLY1" gate="G$1" x="322.58" y="167.64"/>
 <instance part="R40" gate="G$1" x="304.8" y="162.56" rot="R180"/>
 <instance part="R41" gate="G$1" x="297.18" y="154.94" rot="R90"/>
@@
 <instance part="GND21" gate="1" x="12.7" y="149.86"/>
 <instance part="GND22" gate="1" x="12.7" y="132.08"/>
-<instance part="SUPPLY3" gate="G$1" x="63.5" y="180.34"/>
 <instance part="L1" gate="G$1" x="55.88" y="139.7" rot="R180"/>
 <instance part="C21" gate="G$1" x="40.64" y="127"/>
@@
 <instance part="TP5" gate="G$1" x="269.24" y="55.88" rot="R270"/>
 <instance part="TP6" gate="G$1" x="208.28" y="167.64"/>
+<instance part="TP17" gate="G$1" x="104.14" y="208.28"/>
 </instances>
 <busses>
@@
 <segment>
 <pinref part="C15" gate="G$1" pin="1"/>
-<pinref part="R40" gate="G$1" pin="1"/>
-<wire x1="309.88" y1="162.56" x2="312.42" y2="162.56" width="0.1524" layer="91"/>
-<wire x1="312.42" y1="162.56" x2="314.96" y2="162.56" width="0.1524" layer="91"/>
 <wire x1="314.96" y1="162.56" x2="320.04" y2="162.56" width="0.1524" layer="91"/>
 <wire x1="320.04" y1="162.56" x2="320.04" y2="160.02" width="0.1524" layer="91"/>
 <pinref part="IC1" gate="P" pin="V+"/>
 <wire x1="314.96" y1="160.02" x2="314.96" y2="162.56" width="0.1524" layer="91"/>
-<junction x="314.96" y="162.56"/>
 <pinref part="SUPPLY1" gate="G$1" pin="+UB"/>
-<wire x1="312.42" y1="165.1" x2="312.42" y2="162.56" width="0.1524" layer="91"/>
-<junction x="312.42" y="162.56"/>
+<wire x1="322.58" y1="165.1" x2="322.58" y2="162.56" width="0.1524" layer="91"/>
+<wire x1="322.58" y1="162.56" x2="320.04" y2="162.56" width="0.1524" layer="91"/>
+<junction x="320.04" y="162.56"/>
 </segment>
 <segment>
@@
 </segment>
 <segment>
-<pinref part="U$1" gate="G$1" pin="ADVREF"/>
-<pinref part="SUPPLY3" gate="G$1" pin="+UB"/>
-<wire x1="68.58" y1="175.26" x2="63.5" y2="175.26" width="0.1524" layer="91"/>
-<wire x1="63.5" y1="175.26" x2="63.5" y2="177.8" width="0.1524" layer="91"/>
-<pinref part="C26" gate="G$1" pin="2"/>
-<wire x1="60.96" y1="175.26" x2="63.5" y2="175.26" width="0.1524" layer="91"/>
-<junction x="63.5" y="175.26"/>
-</segment>
-<segment>
 <pinref part="SUPPLY4" gate="G$1" pin="+UB"/>
 <wire x1="10.16" y1="198.12" x2="10.16" y2="195.58" width="0.1524" layer="91"/>
@@
 </segment>
 </net>
-<net name="+UB_HALF" class="0">
+<net name="VREF_HALF" class="0">
 <segment>
 <pinref part="IC1" gate="A" pin="+IN"/>
@@
 </segment>
 </net>
-<net name="N$7" class="0">
+<net name="VREF" class="0">
 <segment>
 <pinref part="IC4" gate="G$1" pin="OUT"/>
@@
 <wire x1="208.28" y1="165.1" x2="208.28" y2="162.56" width="0.1524" layer="91"/>
 <junction x="208.28" y="162.56"/>
+<label x="210.82" y="177.8" size="1.27" layer="95" rot="R90"/>
+</segment>
+<segment>
+<pinref part="U$1" gate="G$1" pin="ADVREF"/>
+<wire x1="68.58" y1="175.26" x2="66.04" y2="175.26" width="0.1524" layer="91"/>
+<pinref part="C26" gate="G$1" pin="2"/>
+<wire x1="66.04" y1="175.26" x2="60.96" y2="175.26" width="0.1524" layer="91"/>
+<wire x1="48.26" y1="185.42" x2="66.04" y2="185.42" width="0.1524" layer="91"/>
+<wire x1="66.04" y1="185.42" x2="66.04" y2="175.26" width="0.1524" layer="91"/>
+<junction x="66.04" y="175.26"/>
+<label x="48.514" y="185.674" size="1.27" layer="95"/>
+</segment>
+<segment>
+<pinref part="R40" gate="G$1" pin="1"/>
+<wire x1="309.88" y1="162.56" x2="312.42" y2="162.56" width="0.1524" layer="91"/>
+<wire x1="312.42" y1="162.56" x2="312.42" y2="170.18" width="0.1524" layer="91"/>
+<wire x1="312.42" y1="170.18" x2="320.04" y2="170.18" width="0.1524" layer="91"/>
+<label x="312.42" y="170.688" size="1.27" layer="95"/>
 </segment>
 </net>
@@
 </segment>
 </net>
+<net name="TP17" class="0">
+<segment>
+<pinref part="TP17" gate="G$1" pin="TP"/>
+<pinref part="U$1" gate="G$1" pin="PB8_XOUT"/>
+<wire x1="104.14" y1="205.74" x2="104.14" y2="195.58" width="0.1524" layer="91"/>
+<label x="103.632" y="196.342" size="1.27" layer="95" rot="R90"/>
+</segment>
+</net>
